File: Hardware/Pfeil-backups/Pfeil-2025-01-25_171003/Pfeil.kicad_pcb (KiCad board)
At the start: 4 copper layers, 50 x 6 mm, 62 parts, among them IC1 2536030320001, IC2 nPM1300-CAAA-R, J1 Conn_01x01_Socket, J2 Conn_01x01_Socket, J3 TagConnect, U1 NRF52840-CKAA-R, U2 WSEN-PADS_2511020213301, U3 WSEN-PADS_2511020213301, X1 XTAL 32MHz 8pF, X2 XTAL 32.768kHz 9pF

Commit message: larger pcb
Parts:
- added R10: 4.7k, Resistor_SMD:R_0201_0603Metric, F.Cu at (126.9, 70.5)
- added R11: 4.7k, Resistor_SMD:R_0201_0603Metric, F.Cu at (126.9, 71.8)
- added R14: 4.7k, Resistor_SMD:R_0201_0603Metric, F.Cu at (170.3, 69.0)
- added R15: 4.7k, Resistor_SMD:R_0201_0603Metric, F.Cu at (168.8, 69.0)
- C15: moved to F.Cu
- moved C37 0.12 mm to (153.9, 72.9)
- turned C15 to 180 degrees
Connections:
- C22 pad 1: Net-(U1A-P0.00/XL1) -> Net-(U1C-XC2)
- C33 pad 2: Net-(U1A-P0.00/XL1) -> Net-(U1A-P0.01/XL2)
- U1 pad A2: Net-(U1A-P0.00/XL1) -> Net-(U1C-XC2)
- U1 pad B10: Net-(U1A-P0.00/XL1) -> Net-(U1A-P0.01/XL2)
- X1 pad 2: Net-(U1A-P0.00/XL1) -> Net-(U1C-XC2)
- X2 pad 1: Net-(U1A-P0.00/XL1) -> Net-(U1A-P0.01/XL2)
Routing:
- net /SDA: track 0.00 -> 54.5 mm
- net /SCL: track 0.00 -> 47.3 mm
- net /I2C_SCL: track 79.6 -> 48.5 mm, vias 7 -> 8
- net /I2C_SDA: track 82.6 -> 51.7 mm, vias 6 -> 8
- net /ISDS_INT_00: track 28.3 -> 0.00 mm, vias 5 -> 0
- net /ISDS_INT_01: track 22.5 -> 0.00 mm, vias 3 -> 0
- net Net-(U1A-P0.01/XL2): track 0.00 -> 12.8 mm, vias 0 -> 2
- net Net-(U1A-P0.00/XL1): track 23.0 -> 11.1 mm
- net Net-(U1C-XC2): track 0.00 -> 9.02 mm
- net GND: track 114.4 -> 122.0 mm, vias 21 -> 22
- net VDD: track 22.7 -> 18.3 mm, vias 4 -> 3
- net Net-(U2-SA0): track 2.98 -> 4.59 mm, vias 2 -> 0
- net /SW2: track 6.47 -> 7.33 mm
- net Net-(IC2-SW1): track 2.69 -> 3.51 mm
- net /PADS_INT02: track 30.3 -> 29.6 mm
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