File: Hardware/Pfeil.kicad_pcb (KiCad board)
At the start: 4 copper layers, 50 x 6 mm, 62 parts, among them IC1 2536030320001, IC2 nPM1300-CAAA-R, J1 Conn_01x01_Socket, J2 Conn_01x01_Socket, J3 TagConnect, U1 NRF52840-CKAA-R, U2 WSEN-PADS_2511020213301, U3 WSEN-PADS_2511020213301, X1 XTAL 32MHz 8pF, X2 XTAL 32.768kHz 9pF

Commit message: Fix some shit
Parts:
- removed C26: 1.0pF NPO 5%, Capacitor_SMD:C_0201_0603Metric
- removed L5: 3.9nH 5% 0201, Inductor_SMD:L_0603_1608Metric_Pad1.05x0.95mm_HandSolder
- removed L6: 4.7nH 5% 0201, Inductor_SMD:L_0603_1608Metric_Pad1.05x0.95mm_HandSolder
- added C29: 6.2pF NPO 5%, Capacitor_SMD:C_0201_0603Metric, F.Cu at (132.7, 54.0)
- ANT1, C4, C6: moved to F.Cu
- X2: footprint Crystal:Crystal_SMD_2012-2Pin_2.0x1.2mm -> Crystal:Crystal_SMD_2016-4Pin_2.0x1.6mm
- moved ANT1 18.9 mm to (137.0, 53.0)
- moved C4 18.0 mm to (132.7, 53.2), turned to 0 degrees
- moved X2 17.0 mm to (147.6, 54.7)
- moved C6 16.9 mm to (136.6, 56.0), turned to 0 degrees
- moved X1 15.7 mm to (140.6, 54.1), turned to 90 degrees
- moved C21 15.7 mm to (142.2, 54.9), turned to 90 degrees
- moved C3 15.5 mm to (126.1, 56.5), turned to -90 degrees
- moved C22 15.1 mm to (143.1, 54.9), turned to 90 degrees
- moved R1 15.1 mm to (129.5, 57.0), turned to -90 degrees
- moved L1 14.9 mm to (151.3, 53.8)
- moved U2 14.9 mm to (127.8, 56.4)
- moved C5 14.9 mm to (127.4, 54.8)
- moved C25 14.7 mm to (145.1, 54.9), turned to -90 degrees
- moved C30 14.3 mm to (136.2, 59.2)
- moved C33 14.3 mm to (145.8, 54.9), turned to -90 degrees
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Connections:
- net Net-(ANT1-RADIATOR_ELECTRODE) renamed /RE
- ANT1 pad 2: Net-(ANT1-DUMMY_PAD_1) -> /FEEL
- ANT1 pad 3: Net-(ANT1-DUMMY_PAD_1) -> /FEEL
- ANT1 pad 4: Net-(ANT1-FEED_POINT) -> /FEEL
- C22 pad 1: Net-(U1A-P0.00/XL1) -> Net-(U1C-XC2)
- C33 pad 2: Net-(U1A-P0.00/XL1) -> Net-(U1A-P0.01/XL2)
- C6 pad 1: Net-(ANT1-FEED_POINT) -> GND
- C6 pad 2: /RF -> /FEEL
- U1 pad A2: Net-(U1A-P0.00/XL1) -> Net-(U1C-XC2)
- U1 pad B10: Net-(U1A-P0.00/XL1) -> Net-(U1A-P0.01/XL2)
- U1 pad C9: /I2C_SDA -> unconnected-(U1A-P0.26-PadC9)
- U1 pad E1: Net-(U1A-ANT) -> /FEEL
- U1 pad J5: unconnected-(U1A-P0.20-PadJ5) -> /I2C_SCL
- U1 pad J7: unconnected-(U1A-P0.14-PadJ7) -> /I2C_SDA
- X1 pad 2: Net-(U1A-P0.00/XL1) -> Net-(U1C-XC2)
- X2 pad 1: Net-(U1A-P0.00/XL1) -> Net-(U1A-P0.01/XL2)
Routing:
- net GND: track 114.4 -> 16.9 mm, vias 21 -> 26
- net /I2C_SDA: track 82.6 -> 18.7 mm, vias 6 -> 3
- net +3V3: track 60.0 -> 13.7 mm, vias 3 -> 0
- net /I2C_SCL: track 79.6 -> 53.7 mm
- net /SWDIO: track 25.3 -> 0.00 mm, vias 2 -> 0
- net /SWCLK: track 23.5 -> 2.48 mm
- net Net-(U1A-P0.00/XL1): track 23.0 -> 4.51 mm, vias 3 -> 2
- net /PADS_INT01: track 16.4 -> 0.02 mm, vias 2 -> 1
- net /3.0V: track 11.1 -> 0.00 mm, vias 2 -> 0
- net Net-(ANT1-DUMMY_PAD_1): track 9.63 -> 0.00 mm
- net /FEEL: track 0.00 -> 9.02 mm
- net /PADS_INT02: track 30.3 -> 22.0 mm
- net Net-(U1C-XC1): track 9.41 -> 2.26 mm
- net VDD: track 22.7 -> 17.5 mm, vias 4 -> 2
- net /RF: track 4.95 -> 0.00 mm
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Other:
- board size 50 x 6 mm -> 50 x 9 mm

Commit message: reroute all
Parts:
- removed C20, C35: 10uF X5R 25V 20%, Capacitor_SMD:C_0201_0603Metric
- removed R2: 0R 1%, Resistor_SMD:R_0201_0603Metric
- removed R4, R8: ~, Resistor_SMD:R_0201_0603Metric
- L1, L2: moved to B.Cu
- R1: value 0R 1% -> 100K 1%
- R3: value ~ -> 100K 1%
- moved L2 9.06 mm to (149.8, 54.9), turned to -90 degrees
- moved C30 8.57 mm to (143.6, 54.9), turned to -90 degrees
- moved C7 6.06 mm to (165.1, 55.5)
- moved R9 5.76 mm to (169.5, 59.3), turned to 0 degrees
- moved R5 5.49 mm to (165.1, 56.2), turned to 0 degrees
- moved C8 5.24 mm to (170.3, 54.0), turned to 0 degrees
- moved R6 5.24 mm to (165.1, 56.9), turned to 0 degrees
- moved C3 3.31 mm to (129.4, 57.0)
- moved C9 3.15 mm to (168.3, 54.0), turned to 0 degrees
- moved C1 2.46 mm to (168.3, 54.9)
- moved C2 2.44 mm to (170.3, 57.3), turned to -90 degrees
- moved R3 2.20 mm to (169.4, 58.5)
- moved C15 2.19 mm to (152.6, 55.0), turned to 90 degrees
- moved C12 2.08 mm to (157.1, 56.8), turned to 0 degrees
- moved IC1 1.51 mm to (168.5, 56.7), turned to 0 degrees
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Connections:
- IC2 pad E3: /NRF_SCL -> /I2C_SCL
- IC2 pad E5: /NRF_SDA -> /I2C_SDA
- U1 pad B6: /PADS_INT01 -> unconnected-(U1A-P0.02/AIN0-PadB6)
- U1 pad D9: /I2C_SCL -> unconnected-(U1A-P0.27-PadD9)
- U1 pad J1: unconnected-(U1A-P1.01-PadJ1) -> /PADS_INT01
Routing:
- net /I2C_SDA: track 18.7 -> 47.2 mm
- net /ISDS_INT_00: track 28.3 -> 3.98 mm, vias 4 -> 0
- net /VBAT: track 22.1 -> 0.00 mm, vias 1 -> 0
- net /PADS_INT02: track 22.0 -> 0.00 mm, vias 2 -> 0
- net /RESET: track 17.8 -> 0.00 mm, vias 2 -> 0
- net /PADS_INT01: track 0.02 -> 15.0 mm, vias 1 -> 0
- net GND: track 16.9 -> 31.5 mm, vias 26 -> 34
- net /ISDS_INT_01: track 22.4 -> 9.63 mm, vias 3 -> 1
- net +3V3: track 13.7 -> 6.27 mm
- net /SAO: track 8.93 -> 1.98 mm
- net Net-(IC2-PVDD): track 9.81 -> 3.15 mm, vias 2 -> 0
- net /3.0V: track 0.00 -> 6.09 mm, vias 0 -> 2
- net Net-(U3-SA0): track 2.89 -> 0.00 mm
- net /ISDS_INT: track 4.32 -> 1.77 mm
- net /SWCLK: track 2.48 -> 0.00 mm, vias 2 -> 1
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
Commit message: fixes
Parts:
- moved J1 0.07 mm to (173.4, 56.6)
- moved J2 0.07 mm to (173.4, 56.6)
Connections:
- U1 pad A5: /PADS_INT02 -> unconnected-(U1A-P0.03/AIN1-PadA5)
- U1 pad K7: unconnected-(U1A-P0.15-PadK7) -> /PADS_INT02
Routing:
- net +3V3: track 6.27 -> 89.9 mm, vias 0 -> 4
- net GND: track 31.5 -> 82.5 mm, vias 34 -> 49
- net VDD: track 16.5 -> 63.9 mm, vias 4 -> 9
- net /PADS_INT02: track 0.00 -> 28.6 mm, vias 0 -> 3
- net /SWCLK: track 0.00 -> 27.5 mm, vias 1 -> 2
- net /VBAT: track 0.00 -> 24.2 mm, vias 0 -> 1
- net /ISDS_INT_00: track 3.98 -> 26.9 mm, vias 0 -> 1
- net /ISDS_INT_01: track 9.63 -> 32.1 mm, vias 1 -> 3
- net /SWDIO: track 0.00 -> 20.5 mm, vias 0 -> 2
- net /RESET: track 0.00 -> 18.2 mm
- net Net-(U1B-DEC1): track 7.01 -> 1.11 mm
- net Net-(IC2-PVDD): track 3.15 -> 5.65 mm, vias 0 -> 2
- net /I2C_SCL: track 51.4 -> 49.5 mm
- net Net-(IC2-VOUT1): track 1.96 -> 3.83 mm
- net /FEEL: track 9.02 -> 10.2 mm
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
Commit message: Auf Süüüüüß Puschen
Parts:
- added NT1: NetTie_2, NetTie:NetTie-2_SMD_Pad0.5mm, F.Cu at (138.2, 53.6)
- moved J1 0.23 mm to (173.2, 56.6)
- moved J2 0.23 mm to (173.2, 56.6)
Routing:
- net GND: track 82.5 -> 87.9 mm, vias 49 -> 76
- net /PADS_INT02: track 28.6 -> 26.4 mm
- net +3V3: track 89.9 -> 88.3 mm

Commit message: fixing and routing
Parts:
- added C26: 1pF 5% 0201, Capacitor_SMD:C_0201_0603Metric, F.Cu at (139.3, 57.0)
- added L3: 3.9nH 0201 5%, Inductor_SMD:L_0201_0603Metric, F.Cu at (140.4, 57.3)
- added L4: 4.7nH 0201 5%, Inductor_SMD:L_0201_0603Metric, F.Cu at (138.3, 57.3)
- added R10: 1K 1%, Resistor_SMD:R_0201_0603Metric, F.Cu at (166.9, 56.6)
- added R8: 1K 1%, Resistor_SMD:R_0201_0603Metric, F.Cu at (167.9, 58.3)
- C12, C13, C14, C15, C16, C19, C2, C36, C5: footprint Capacitor_SMD:C_0201_0603Metric -> Capacitor_SMD:C_0402_1005Metric
- L1, L2: footprint Inductor_SMD:L_0603_1608Metric_Pad1.05x0.95mm_HandSolder -> Inductor_SMD:L_0201_0603Metric
- moved L2 0.97 mm to (150.6, 55.4)
- moved L1 0.63 mm to (151.6, 55.4)
- moved C13 0.49 mm to (157.2, 55.6)
- moved C19 0.38 mm to (154.5, 54.9)
- moved C12 0.26 mm to (157.2, 56.6)
- moved C16 0.20 mm to (153.5, 54.9)
- moved C14 0.11 mm to (157.2, 57.5)
- moved R3 0.09 mm to (169.4, 58.6)
- moved C5 0.09 mm to (127.4, 54.7)
- moved C15 0.06 mm to (152.6, 54.9)
- moved C36 0.05 mm to (151.2, 57.3)
Connections:
- IC1 pad 1: /SAO -> VDD
- IC1 pad 14: /I2C_SDA -> /I2C_SCL
- IC1 pad 2: /RSVD3 -> VDD
- IC1 pad 3: /RSVD2 -> VDD
- IC1 pad 4: /ISDS_INT_00 -> VDD
- IC2 pad E5: /I2C_SDA -> /I2C_SCL
- R5 pad 2: /RSVD2 -> VDD
- R6 pad 2: /RSVD3 -> VDD
- R7 pad 2: /SAO -> VDD
- U1 pad C10: /ISDS_INT_00 -> VDD
- U1 pad E1: /FEEL -> Net-(U1A-ANT)
- U1 pad J7: /I2C_SDA -> /I2C_SCL
- U2 pad 4: /I2C_SDA -> /I2C_SCL
- U3 pad 4: /I2C_SDA -> /I2C_SCL
Routing:
- net /I2C_SCL: track 49.5 -> 99.2 mm, vias 4 -> 7
- net /I2C_SDA: track 47.7 -> 0.00 mm, vias 3 -> 0
- net VDD: track 63.9 -> 99.2 mm, vias 9 -> 10
- net /ISDS_INT_00: track 27.0 -> 0.00 mm, vias 1 -> 0
- net GND: track 87.9 -> 93.8 mm, vias 76 -> 73
- net /VBAT: track 24.2 -> 19.5 mm, vias 1 -> 2
- net /FEEL: track 10.2 -> 6.20 mm
- net /RSVD2: track 2.02 -> 0.00 mm
- net /SAO: track 1.98 -> 0.00 mm
- net /RSVD3: track 1.93 -> 0.00 mm
- net Net-(U1A-ANT): track 0.00 -> 1.66 mm
- net Net-(C26-Pad1): track 0.00 -> 1.53 mm
- net /3.0V: track 6.90 -> 5.45 mm
- net Net-(IC2-VOUT1): track 4.02 -> 3.19 mm
- net +3V3: track 88.3 -> 88.9 mm
