File: Hardware/Pfeil.kicad_pcb (KiCad board)
At the start: 4 copper layers, 50 x 13 mm, 52 parts, among them IC1 2536030320001, IC2 AP7312-1233FM-7, J1 Conn_01x01_Pin, J2 Conn_01x01_Pin, J3 TagConnect, U2 WSEN-PADS_2511020213301, U3 WSEN-PADS_2511020213301, U4 nRF52840, X1 XTAL 32MHz 8pF, X2 XTAL 32.768kHz 9pF

Commit message: final
Parts:
- moved C43 1.55 mm to (143.1, 52.9), turned to 0 degrees
- moved C40 0.23 mm to (141.2, 53.0)
- moved C47 0.16 mm to (138.0, 53.0)
- moved X1 0.12 mm to (134.8, 53.6)
- moved NT1 0.11 mm to (153.8, 53.0)
Routing:
- net Net-(U4-DEC6): track 1.84 -> 3.26 mm
- net GND: track 25.6 -> 26.4 mm, vias 80 -> 83
Other:
- board text added: "APS1"
- board text added: "APS2"
- board text added: "IMU1"
- board text added: "supported by Mardu"
