File: Hardware/Pfeil.kicad_sch (KiCad schematic)
At the start: 66 parts, among them IC1 2536030320001, IC2 nPM1300-CAAA-R, J1 Conn_01x01_Socket, J2 Conn_01x01_Socket, J3 TagConnect, U1 NRF52840-CKAA-R, U2 WSEN-PADS_2511020213301, U3 WSEN-PADS_2511020213301, X1 XTAL 32MHz 8pF, X2 XTAL 32.768kHz 9pF

Commit message: first changes
Parts:
- removed R10, R11, R14, R15: 4.7k, Resistor_SMD:R_0201_0603Metric, symbol Device:R
Connections:
- net SCL is gone; now on net I2C_SCL: IC1.13 (SCL), U1.D9 (P0.27)
- net SDA is gone; now on net I2C_SDA: IC1.14 (SDA), U1.C9 (P0.26)
- net PADS_INT01: no longer U1.A5 (P0.03/AIN1), U3.7 (INT_DRDY)
- new net PADS_INT02: U1.A5 (P0.03/AIN1), U3.7 (INT_DRDY)

Commit message: bezeichner update
Connections:
- net INT_0 is gone; now on net ISDS_INT_00: IC1.4 (INT_0)
- net INT_1 is gone; now on net ISDS_INT_01: IC1.9 (INT_1)
- net ISDS_INT_00: now reaches U1.C10 (P0.04/AIN2)
- net ISDS_INT_01: now reaches U1.D10 (P0.05/AIN3)
- net CS renamed ISDS_INT
- no-connect marks 9 -> 50
Other:
- note added: "Crystal for NRF"
- note added: "NRF52840"
- note added: "Supply for NRF"
- moved on the sheet: ANT1, C1, C10, C11, C12, C13, C14, C15, C16, C17, C18, C19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

Commit message: Fix some shit
Parts:
- removed C26: 1.0pF NPO 5%, Capacitor_SMD:C_0201_0603Metric, symbol Device:C
- removed L5: 3.9nH 5% 0201, Inductor_SMD:L_0603_1608Metric_Pad1.05x0.95mm_HandSolder, symbol Device:L
- removed L6: 4.7nH 5% 0201, Inductor_SMD:L_0603_1608Metric_Pad1.05x0.95mm_HandSolder, symbol Device:L
- added C29: 6.2pF NPO 5%, Capacitor_SMD:C_0201_0603Metric, symbol Device:C
- X1: MFR (none) -> Q22FA12800025
- X2: footprint Crystal:Crystal_SMD_2012-2Pin_2.0x1.2mm -> Crystal:Crystal_SMD_2016-4Pin_2.0x1.6mm; MFR (none) -> 7E032768H01
Connections:
- net RF is gone; now on net FEEL: C6.2
- net GND: now also C6.1, C29.2
- net FEEL: now reaches ANT1.2 (DUMMY_PAD_1), ANT1.3 (DUMMY_PAD_2)
- net FEEL: now also ANT1.4 (FEED_POINT), U1.E1 (ANT)
- net RE: now reaches ANT1.1 (RADIATOR_ELECTRODE), C4.2
- net RE: now also C29.1
Other:
- moved on the sheet: ANT1, C4, C6, J3, X2

Commit message: reroute all
Parts:
- removed R8: ~, Resistor_SMD:R_0201_0603Metric, symbol Device:R
- C20, C35, R2: now not fitted; now left out of the parts list
- R1: value 0R 1% -> 100K 1%
- R3: value ~ -> 100K 1%; now fitted
- R4: now left out of the parts list
Connections:
- net NRF_SCL is gone; now on net I2C_SCL: IC2.E3 (SCL)
- net NRF_SDA is gone; now on net I2C_SDA: IC2.E5 (SDA)
- net I2C_SCL: now also U1.J5 (P0.20); no longer U1.D9 (P0.27)
- net I2C_SDA: now also U1.J7 (P0.14); no longer U1.C9 (P0.26)
- net PADS_INT01: now also U1.J1 (P1.01); no longer U1.B6 (P0.02/AIN0)
- no-connect marks 50 -> 47

Commit message: fixes
Connections:
- net PADS_INT02: now also U1.K7 (P0.15); no longer U1.A5 (P0.03/AIN1)
Changed lines of the file:
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@@
 	)
 	(no_connect
-		(at 67.31 77.47)
+		(at 67.31 46.99)
 	)
 	(no_connect
@@
 	(wire
 		(pts
+			(xy 53.34 77.47) (xy 67.31 77.47)
+		)
+		(stroke
+			(width 0)
+			(type default)
+		)
+	)
+	(wire
+		(pts
 			(xy 288.29 115.57) (xy 297.18 115.57)
 		)
@@
 		(pts
 			(xy 314.96 182.88) (xy 314.96 185.42)
-		)
-		(stroke
-			(width 0)
-			(type default)
-		)
-	)
-	(wire
-		(pts
-			(xy 53.34 46.99) (xy 67.31 46.99)
 		)
 		(stroke
@@
 	)
 	(label "PADS_INT02"
-		(at 53.34 46.99 0)
-		(fields_autoplaced yes)
-		(effects
+		(at 53.34 77.47 0)
+		(fields_autoplaced yes)
+		(effects

Commit message: Auf Süüüüüß Puschen
Parts:
- added NT1: NetTie_2, NetTie:NetTie-2_SMD_Pad0.5mm, symbol Device:NetTie_2
Connections:
- net FEEL: now also NT1.2
- net GND: now also NT1.1
Changed lines of the file:
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@@
 	(wire
 		(pts
+			(xy 149.86 24.13) (xy 152.4 24.13)
+		)
+		(stroke
+			(width 0)
+			(type default)
+		)
+	)
+	(wire
+		(pts
 			(xy 130.81 242.57) (xy 123.19 242.57)
 		)
@@
 	(wire
 		(pts
+			(xy 157.48 24.13) (xy 163.83 24.13)
+		)
+		(stroke
+			(width 0)
+			(type default)
+		)
+	)
+	(wire
+		(pts
 			(xy 180.34 217.17) (xy 180.34 219.71)
 		)
@@
 		)
 	)
+	(label "FEEL"
+		(at 163.83 24.13 180)
+		(fields_autoplaced yes)
+		(effects
+			(font
+				(size 1.27 1.27)
+			)
+			(justify right bottom)
+		)
+	)
 	(label "RE"
 		(at 156.21 50.8 0)
@@
 	)
 	(symbol
+		(lib_id "power:GND")
+		(at 149.86 24.13 270)
+		(unit 1)
+		(exclude_from_sim no)
+		(in_bom yes)
+		(on_board yes)
+		(dnp no)
+		(property "Reference" "#PWR017"
+			(at 143.51 24.13 0)
+			(effects
+				(font
+					(size 1.27 1.27)
+				)
+				(hide yes)
+			)
+		)
+		(property "Value" "GND"
+			(at 144.526 26.162 0)
+			(effects
+				(font
+					(size 1.27 1.27)
+				)
+				(justify right)
+			)
+		)
+		(property "Footprint" ""
+			(at 149.86 24.13 0)
+			(effects
+				(font
+					(size 1.27 1.27)
+				)
+				(hide yes)
+			)
+		)
+		(property "Datasheet" ""
+			(at 149.86 24.13 0)
+			(effects
+				(font
+					(size 1.27 1.27)
+				)
+				(hide yes)
+			)
+		)
+		(property "Description" "Power symbol creates a global label with name \"GND\" , ground"
+			(at 149.86 24.13 0)
+			(effects
+				(font
+					(size 1.27 1.27)
+				)
+				(hide yes)
+			)
+		)
+		(pin "1"
+		)
+		(instances
+			(project "Pfeil"
+				(path "/6779a91c-36f7-4406-b6b7-047f6d9775a9"
+					(reference "#PWR017")
+					(unit 1)
+				)
+			)
+		)
+	)
+	(symbol
 		(lib_id "Device:C")
 		(at 382.27 45.72 180)
@@
 					(unit 1)
 				)
+			)
+		)
+	)
+	(symbol
+		(lib_id "Device:NetTie_2")
+		(at 154.94 24.13 0)
+		(unit 1)
+		(exclude_from_sim no)
+		(in_bom no)
+		(on_board yes)
+		(dnp no)
+		(fields_autoplaced yes)
+		(property "Reference" "NT1"
+			(at 154.94 19.05 0)
+			(effects
+				(font
+					(size 1.27 1.27)
+				)
+			)
+		)
+		(property "Value" "NetTie_2"
+			(at 154.94 21.59 0)
+			(effects
+				(font
+					(size 1.27 1.27)
+				)
+			)
+		)
+		(property "Footprint" "NetTie:NetTie-2_SMD_Pad0.5mm"
+			(at 154.94 24.13 0)
+			(effects
+				(font
+					(size 1.27 1.27)
+				)
+				(hide yes)
+			)
+		)
+		(property "Datasheet" "~"
+			(at 154.94 24.13 0)
+			(effects
+				(font
+					(size 1.27 1.27)
+				)
+				(hide yes)
+			)
+		)
+		(property "Description" "Net tie, 2 pins"
+			(at 154.94 24.13 0)
+			(effects
+				(font
+					(size 1.27 1.27)
+				)
+				(hide yes)
+			)
+		)
+		(pin "1"
+		)
+		(pin "2"
+		)
+		(instances
+			(project ""
+				(path "/6779a91c-36f7-4406-b6b7-047f6d9775a9"
+					(reference "NT1")
+					(unit 1)
+				)

Commit message: fixing and routing
Parts:
- added C26: 1pF 5% 0201, Capacitor_SMD:C_0201_0603Metric, symbol Device:C
- added L3: 3.9nH 0201 5%, Inductor_SMD:L_0201_0603Metric, symbol Device:L
- added L4: 4.7nH 0201 5%, Inductor_SMD:L_0201_0603Metric, symbol Device:L
- added R10, R8: 1K 1%, Resistor_SMD:R_0201_0603Metric, symbol Device:R
- C12, C13, C14, C15, C16, C19, C2, C36, C5: footprint Capacitor_SMD:C_0201_0603Metric -> Capacitor_SMD:C_0402_1005Metric
- L1, L2: footprint Inductor_SMD:L_0603_1608Metric_Pad1.05x0.95mm_HandSolder -> Inductor_SMD:L_0201_0603Metric
Connections:
- net I2C_SDA is gone; now on net I2C_SCL: IC1.14 (SDA), IC2.E5 (SDA), U1.J7 (P0.14), U2.4 (SDA), U3.4 (SDA)
- net ISDS_INT_00 is gone; now on net VDD: IC1.4 (INT_0), U1.C10 (P0.04/AIN2)
- net RSVD2 is gone; now on net VDD: IC1.3 (RSVD_2), R5.2
- net RSVD3 is gone; now on net VDD: IC1.2 (RSVD_1), R6.2
- net SAO is gone; now on net VDD: IC1.1 (SAO), R7.2
- net FEEL: now also L4.2; no longer U1.E1 (ANT)
- net GND: now also C26.2, R10.1, R8.1
- net I2C_SCL: now also R10.2, R8.2
- new net: L3.1, U1.E1 (ANT)
- new net: C26.1, L3.2, L4.1
Other:
- moved on the sheet: ANT1, C17, C18, C23, C24, C25, C27, C28, C29, C30, C31, C34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

Commit message: nrf 52840 changing of the package
Parts:
- removed C17, C18: 1uF X7R 10%, Capacitor_SMD:C_0201_0603Metric, symbol Device:C
- removed C21, C22: 12pF NP0 2%, Capacitor_SMD:C_0201_0603Metric, symbol Device:C
- removed C23, C24, C31: 4.7uF X7R 10%, Capacitor_SMD:C_0201_0603Metric, symbol Device:C
- removed C25, C28, C30: 100nF X7R 10%, Capacitor_SMD:C_0201_0603Metric, symbol Device:C
- removed C26: 1pF 5% 0201, Capacitor_SMD:C_0201_0603Metric, symbol Device:C
- removed C27: 4.7uF X7S 10%, Capacitor_SMD:C_0201_0603Metric, symbol Device:C
- removed C34: 820pF X7R 10%, Capacitor_SMD:C_0201_0603Metric, symbol Device:C
- removed L3: 3.9nH 0201 5%, Inductor_SMD:L_0201_0603Metric, symbol Device:L
- removed L4: 4.7nH 0201 5%, Inductor_SMD:L_0201_0603Metric, symbol Device:L
- removed U1: NRF52840-CKAA-R, NRF52840-CKAA-R:BGA94C35P10X10_360X354X51N, symbol NRF52840-CKAA-R:NRF52840-CKAA-R
- removed X1: XTAL 32MHz 8pF, Crystal:Crystal_SMD_2016-4Pin_2.0x1.6mm, symbol Device:Crystal
- added C38, C49, C50, C51: 100nF, Capacitor_SMD:C_0201_0603Metric, symbol Device:C
- added C39, C43: N.C., Capacitor_SMD:C_0201_0603Metric, symbol Device:C
- added C40: 100pF, Capacitor_SMD:C_0201_0603Metric, symbol Device:C
- added C41: 1pF, Capacitor_SMD:C_0201_0603Metric, symbol Device:C
- added C42, C45: 820pF, Capacitor_SMD:C_0201_0603Metric, symbol Device:C
- added C44, C46: 4.7uF, Capacitor_SMD:C_0201_0603Metric, symbol Device:C
- added C47, C48: 12pF NP0 2%, Capacitor_SMD:C_0201_0603Metric, symbol Device:C
- added L5: L, Inductor_SMD:L_0201_0603Metric, symbol Device:L
- added R11: 2R2, Resistor_SMD:R_0201_0603Metric, symbol Device:R
- added U4: nRF52840, Package_DFN_QFN:Nordic_AQFN-73-1EP_7x7mm_P0.5mm, symbol MCU_Nordic:nRF52840
- added X3: XTAL 32MHz 8pF, Crystal:Crystal_SMD_2016-4Pin_2.0x1.6mm, symbol Device:Crystal
Connections:
- net GND: now also C38.1, C39.1, C40.1, C41.1, C42.1, C43.2, C44.1, C45.2, C46.1, C47.2, C48.2, C49.2, C50.2, C51.2, U4.B7 (VSS), U4.EP (VSS), U4.F23 (VSS_PA)
- net at X2.2: now also C33.2, U4.D2 (XL1/P0.00); no longer C32.1
- net at X2.1: now also C32.1, U4.F2 (XL2/P0.01); no longer C33.2
- net VDD renamed ISDS_INT_00
- new net: C39.2, U4.A18 (DEC2)
- new net: C48.1, U4.A23 (XC2), X3.2
- new net: C44.2, U4.AC5 (DECUSB)
- new net: C47.1, U4.B24 (XC1), X3.1
- new net: C41.2, U4.B5 (DEC4)
- new net: C38.2, U4.C1 (DEC1)
- new net: C40.2, U4.D23 (DEC3)
- new net: C43.1, U4.E24 (DEC6)
- new net: C49.1, L5.2, U4.H23 (ANT)
- new net: C42.2, U4.N24 (DEC5)
- new net: C50.1, C51.1, L5.1
- new net D+: U4.AD6 (D+)
- new net D-: U4.AD4 (D-)
- new net GND VBUS: R11.2
- new net GND VBUS NRF: C45.1, R11.1, U4.AD2 (VBUS), U4.Y2 (VDDH)
- new net GND VDD NRF: C46.2, U4.A22 (VDD), U4.AD14 (VDD), U4.AD23 (VDD), U4.B1 (VDD), U4.W1 (VDD)
- no-connect marks 47 -> 59
Other:
- note removed: "Crystal for NRF"
- note removed: "NRF52840"
- note removed: "Supply for NRF"
- moved on the sheet: C32, C33, X2
