File: Hardware/Pfeil.kicad_sch (KiCad schematic)
At the start: 66 parts, among them IC1 2536030320001, IC2 nPM1300-CAAA-R, J1 Conn_01x01_Socket, J2 Conn_01x01_Socket, J3 TagConnect, U2 WSEN-PADS_2511020213301, U3 WSEN-PADS_2511020213301, U4 nRF52840, X2 XTAL 32.768kHz 9pF, X3 XTAL 32MHz 8pF

Commit message: bigger pcb and no more npm1300
Parts:
- removed C10: 1.0uF, Capacitor_SMD:C_0201_0603Metric, symbol Device:C
- removed C11: 1.0uF X5R 10V 10%, Capacitor_SMD:C_0201_0603Metric, symbol Device:C
- removed C12, C13, C14, C15, C16, C19, C36: 10uF X5R 25V 20%, Capacitor_SMD:C_0402_1005Metric, symbol Device:C
- removed C20, C35: 10uF X5R 25V 20%, Capacitor_SMD:C_0201_0603Metric, symbol Device:C
- removed C37: 100nF X5R 10%, Capacitor_SMD:C_0201_0603Metric, symbol Device:C
- removed IC2: nPM1300-CAAA-R, nPM1300-CAAA-R:BGA35C44P7X5_308X238X51, symbol nPM1300-CAAA-R:nPM1300-CAAA-R
- removed J1, J2: Conn_01x01_Socket, TestPoint:TestPoint_Pad_2.5x2.5mm, symbol Connector:Conn_01x01_Socket
- removed L1, L2: 2.2uH DCR <400mR 20%, Inductor_SMD:L_0201_0603Metric, symbol Device:L
- removed R12: 47k 1%, Resistor_SMD:R_0201_0603Metric, symbol Device:R
- removed R13: 270k 1%, Resistor_SMD:R_0201_0603Metric, symbol Device:R
Connections:
- net GND VBUS is gone; now on net GND: R11.2
- net GND VDD NRF is gone; now on net GND: C46.2, U4.A22 (VDD), U4.AD14 (VDD), U4.AD23 (VDD), U4.B1 (VDD), U4.W1 (VDD)
- no-connect marks 59 -> 50
Other:
- moved on the sheet: C1, C2, C3, C32, C33, C38, C39, C40, C41, C42, C43, C44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

Commit message: start ing to routing with the new pcb
Parts:
- added C10, C11, C12: 1uF, Capacitor_SMD:C_0201_0603Metric, symbol Device:C
- added IC2: AP7312-1233FM-7, LIB_AP7312-1233FM-7:SON50P201X181X60-7N, symbol AP7312-1233FM-7:AP7312-1233FM-7
Connections:
- net FEEL: now also C50.1, C51.1, L5.1
- net GND: now also C10.2, C11.2, C12.2, IC2.4 (GND), IC2.7 (EP)
- net I2C_SCL: no longer IC1.13 (SCL), IC1.14 (SDA), R8.2, U2.2 (SCL), U2.4 (SDA), U3.2 (SCL), U3.4 (SDA)
- net RESET: now also U4.AC13 (P0.18/~{RESET})
- net SWCLK: now also U4.AA24 (SWDCLK)
- net SWDIO: now also U4.AC24 (SWDIO)
- net I2C_SDA : now reaches U4.AC21 (P0.25)
- net I2C_SDA : now also U2.4 (SDA), U3.4 (SDA)
- net I2C_SCL : now reaches U4.G1 (P0.26)
- net I2C_SCL : now also IC1.13 (SCL), U2.2 (SCL), U3.2 (SCL)
- new net: C10.1, IC2.5 (OUT2)
- new net: C12.1, IC2.3 (EN2)
- new net: C11.1, IC2.6 (OUT1)
- new net I2C_SDA: IC1.14 (SDA), R8.2
- no-connect marks 50 -> 46
Other:
- moved on the sheet: ANT1, C1, C2, C29, C3, C32, C33, C38, C39, C4, C40, C41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

Commit message: Routing and evry component is on the front
Connections:
- net I2C_SCL is gone; now on net I2C_SCL : R10.2
- net +3V3: now also C10.2, C46.2, C8.1, C9.1, IC1.8 (VDD), IC2.4 (GND), U4.A22 (VDD), U4.AD14 (VDD), U4.AD23 (VDD), U4.B1 (VDD), U4.W1 (VDD)
- net GND: no longer C10.2, C46.2, IC2.4 (GND), U4.A22 (VDD), U4.AD14 (VDD), U4.AD23 (VDD), U4.B1 (VDD), U4.W1 (VDD)
- net I2C_SCL : now also U4.U1 (TRACEDATA1/P0.12); no longer U2.2 (SCL), U3.2 (SCL), U4.G1 (P0.26)
- net I2C_SDA: now also U4.AD8 (P0.13)
- net ISDS_INT_00: no longer C8.1, C9.1, IC1.8 (VDD)
- net I2C_SCL A2: now reaches U4.A12 (AIN0/P0.02)
- net I2C_SCL A2: now also U3.2 (SCL)
- net I2C_SDA A2: now reaches U4.B13 (AIN1/P0.03)
- net I2C_SDA A2: now also U3.4 (SDA)
- net I2C_SDA  renamed I2C_SDA A1
- net I2C_SDA A1: no longer U3.4 (SDA)
- new net I2C_SCL A1: U2.2 (SCL), U4.G1 (P0.26)
- no-connect marks 46 -> 41

Commit message: Luca Berthold review
Parts:
- removed X3: XTAL 32MHz 8pF, Crystal:Crystal_SMD_2016-4Pin_2.0x1.6mm, symbol Device:Crystal
- added X1: XTAL 32MHz 8pF, Crystal:Crystal_SMD_2016-4Pin_2.0x1.6mm, symbol Device:Crystal
Connections:
- net ISDS_INT: now also R9.2; no longer R9.1
- net ISDS_INT_00: no longer C7.1, IC1.1 (SAO), IC1.2 (RSVD_1), IC1.3 (RSVD_2), IC1.5 (VDD_IO), R5.1, R5.2, R6.1, R6.2, R7.1, R7.2, R9.2
- net at C48.1, U4.A23 (XC2): now also X1.1
- net at C47.1, U4.B24 (XC1): now also X1.2
- net RSVD0: no longer names the net of IC1.10 (RSVD_3)
- net RSVD1: no longer names the net of IC1.11 (RSVD_4)
- new net RSVD2: IC1.3 (RSVD_2), R5.2
- new net RSVD3: IC1.2 (RSVD_1), R6.2
- new net SAO: IC1.1 (SAO), R7.2
- new net VDD_IO: C7.1, IC1.5 (VDD_IO), R5.1, R6.1, R7.1, R9.1
- no-connect marks 41 -> 43
Other:
- moved on the sheet: R10, R6, R7, R8, R9

Commit message: Bestellte version
Parts:
- added C13: 1uF, Capacitor_SMD:C_0805_2012Metric, symbol Device:C
- added J1, J2: Conn_01x01_Pin, Connector_Wire:SolderWirePad_1x01_SMD_1x2mm, symbol Connector:Conn_01x01_Pin
- C10, C11, C12: footprint Capacitor_SMD:C_0201_0603Metric -> Capacitor_SMD:C_0805_2012Metric
- C49: value 100nF -> N.C.; now not fitted
- C50: value 100nF -> 0.5pF NPO +10%
- C51: value 100nF -> 0.8pF NPO +10%
- L5: value L -> 4.7nH 5% HF; footprint Inductor_SMD:L_0201_0603Metric -> LED_SMD:LED_0402_1005Metric
Connections:
- net GND: now also C13.2, J2.1 (Pin_1)
- net ISDS_INT_00: now also U4.AD16 (P0.20)
- net ISDS_INT_01: now also U4.AD18 (P0.22)
- net at IC2.1 (IN): now also C13.1, J1.1 (Pin_1)
- no-connect marks 43 -> 40

Commit message: update last
Changed lines of the file:
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@@
 (kicad_sch
-	(version 20231120)
+	(version 20250114)
 	(generator "eeschema")
-	(generator_version "8.0")
+	(generator_version "9.0")
 	(paper "A3")
+	(text "TagConnect Header"
+		(exclude_from_sim no)
+		(at 105.41 220.98 0)
+		(effects
+			(font
+				(size 2.54 2.54)
+			)
+			(justify left bottom)
+		)
+	)
 	(junction
 		(at 128.27 148.59)
@@
 	)
 	(junction
+		(at 364.49 41.91)
+		(diameter 0)
+		(color 0 0 0 0)
+	)
+	(junction
 		(at 148.59 156.21)
 		(diameter 0)
@@
 	)
 	(junction
-		(at 364.49 46.99)
-		(diameter 0)
-		(color 0 0 0 0)
-	)
-	(junction
 		(at 229.87 77.47)
 		(diameter 0)
@@
 	(wire
 		(pts
-			(xy 364.49 46.99) (xy 381 46.99)
+			(xy 364.49 41.91) (xy 381 41.91)
 		)
 		(stroke
@@
 	(wire
 		(pts
-			(xy 381 60.96) (xy 381 46.99)
+			(xy 381 60.96) (xy 381 41.91)
 		)
 		(stroke
@@
 	(wire
 		(pts
-			(xy 364.49 46.99) (xy 364.49 41.91)
-		)
-		(stroke
-			(width 0)
-			(type default)
-		)
-	)
-	(wire
-		(pts
 			(xy 391.16 170.18) (xy 391.16 172.72)
 		)
@@
 	(wire
 		(pts
-			(xy 364.49 48.26) (xy 364.49 46.99)
+			(xy 364.49 41.91) (xy 364.49 48.26)
 		)
 		(stroke
@@
 		)
 	)
-	(text "TagConnect Header"
-		(exclude_from_sim no)
-		(at 105.41 220.98 0)
-		(effects
-			(font
-				(size 2.54 2.54)
-			)
-			(justify left bottom)
-		)
-	)
 	(label "I2C_SDA A2"
 		(at 240.03 138.43 180)
-		(fields_autoplaced yes)
 		(effects
 			(font
@@
 	(label "RF"
 		(at 132.08 109.22 0)
-		(fields_autoplaced yes)
 		(effects
 			(font
@@
 	(label "FEEL"
 		(at 127 100.33 0)
-		(fields_autoplaced yes)
 		(effects
 			(font
@@
 	(label "ISDS_INT_00"
 		(at 317.5 158.75 0)
-		(fields_autoplaced yes)
 		(effects
 			(font
@@
 	(label "I2C_SCL "
 		(at 229.87 161.29 0)
-		(fields_autoplaced yes)
 		(effects
 			(font
@@
 	(label "RESET"
 		(at 116.84 231.14 90)
-		(fields_autoplaced yes)
 		(effects
 			(font
@@
 	(label "I2C_SDA A2"
 		(at 398.78 53.34 180)
-		(fields_autoplaced yes)
 		(effects
 			(font
@@
 	(label "I2C_SDA A1"
 		(at 318.77 53.34 180)
-		(fields_autoplaced yes)
 		(effects
 			(font
@@
 	(label "RSVD2"
 		(at 347.98 156.21 0)
-		(fields_autoplaced yes)
 		(effects
 			(font
@@
 	(label "I2C_SCL "
 		(at 372.11 127 270)
-		(fields_autoplaced yes)
 		(effects
 			(font
@@
 	(label "PADS_INT02"
 		(at 392.43 66.04 180)
-		(fields_autoplaced yes)
 		(effects
 			(font
@@
 	(label "RF"
 		(at 107.95 148.59 0)
-		(fields_autoplaced yes)
 		(effects
 			(font
@@
 	(label "SWDIO"
 		(at 124.46 231.14 90)
-		(fields_autoplaced yes)
 		(effects
 			(font
@@
 	(label "SAO"
 		(at 347.98 151.13 0)
-		(fields_autoplaced yes)
 		(effects
 			(font
@@
 	(label "D-"
 		(at 234.95 255.27 0)
-		(fields_autoplaced yes)
 		(effects
 			(font
@@
 	(label "ISDS_INT_01"
 		(at 241.3 184.15 180)
-		(fields_autoplaced yes)
 		(effects
 			(font
@@
 	(label "VDD"
 		(at 405.13 158.75 180)
-		(fields_autoplaced yes)
 		(effects
 			(font
@@
 	(label "RESET"
 		(at 162.56 237.49 180)
-		(fields_autoplaced yes)
 		(effects
 			(font
@@
 	(label "SWCLK"
 		(at 121.92 231.14 90)
-		(fields_autoplaced yes)
 		(effects
 			(font
@@
 	(label "I2C_SCL A1"
 		(at 318.77 58.42 180)
-		(fields_autoplaced yes)
 		(effects
 			(font
@@
 	(label "RSVD3"
 		(at 347.98 153.67 0)
-		(fields_autoplaced yes)
 		(effects
 			(font
@@
 	(label "ISDS_INT_01"
 		(at 405.13 156.21 180)
-		(fields_autoplaced yes)
 		(effects
 			(font
@@
 	(label "FEEL"
 		(at 99.06 129.54 90)
-		(fields_autoplaced yes)
 		(effects
 			(font
@@
 	(label "VDD_IO"
 		(at 317.5 138.43 0)
-		(fields_autoplaced yes)
 		(effects
 			(font
@@
 	(label "FEEL"
 		(at 99.06 71.12 270)
-		(fields_autoplaced yes)
 		(effects
 			(font
@@
 	(label "ISDS_INT"
 		(at 374.65 127 270)
-		(fields_autoplaced yes)
 		(effects
 			(font
@@
 	(label "SWDIO"
 		(at 162.56 242.57 180)
-		(fields_autoplaced yes)
 		(effects
 			(font
@@
 	(label "I2C_SCL A2"
 		(at 398.78 58.42 180)
-		(fields_autoplaced yes)
 		(effects
 			(font
@@
 	(label "SWO"
 		(at 127 231.14 90)
-		(fields_autoplaced yes)
 		(effects
 			(font
@@
 	(label "SWCLK"
 		(at 162.56 240.03 180)
-		(fields_autoplaced yes)
 		(effects
 			(font
@@
 	(label "I2C_SDA"
 		(at 229.87 163.83 0)
-		(fields_autoplaced yes)
 		(effects
 			(font
@@
 	(label "I2C_SDA"
 		(at 369.57 128.27 270)
-		(fields_autoplaced yes)
 		(effects
 			(font
@@
 	(label "VDD_IO"
 		(at 393.7 127 180)
-		(fields_autoplaced yes)
 		(effects
 			(font
@@
 	(label "I2C_SCL A1"
 		(at 240.03 194.31 180)
-		(fields_autoplaced yes)
 		(effects
 			(font
@@
 	(label "PADS_INT01"
 		(at 312.42 66.04 180)
-		(fields_autoplaced yes)
 		(effects
 			(font
@@
 	(label "I2C_SCL A2"
 		(at 240.03 135.89 180)
-		(fields_autoplaced yes)
 		(effects
 			(font
@@
 	(label "VDD_IO"
 		(at 369.57 195.58 90)
-		(fields_autoplaced yes)
 		(effects
 			(font
@@
 	(label "D+"
 		(at 234.95 257.81 0)
-		(fields_autoplaced yes)
 		(effects
 			(font
@@
 	(label "I2C_SDA A1"
 		(at 240.03 191.77 180)
-		(fields_autoplaced yes)
 		(effects
 			(font
@@
 	(label "I2C_SCL "
 		(at 374.65 107.95 270)
-		(fields_autoplaced yes)
 		(effects
 			(font
@@
 	(label "FEEL"
 		(at 76.2 72.39 180)
-		(fields_autoplaced yes)
 		(effects
 			(font
@@
 	(label "RE"
 		(at 66.04 99.06 0)
-		(fields_autoplaced yes)
 		(effects
 			(font
@@
 	(label "I2C_SDA"
 		(at 361.95 107.95 270)
-		(fields_autoplaced yes)
 		(effects
 			(font
@@
 	(label "ISDS_INT_00"
 		(at 241.3 179.07 180)
-		(fields_autoplaced yes)
 		(effects
 			(font
@@
 		)
 	)
+	(embedded_fonts no)
 )
